Commit message: Attempt to get 2 robotarms in one gazebo simulation
Parametrize transmission, joint and actuator names by the robotname.
In the urdf, spawn 2 iiwas, one called iiwa, one called iiwa2.
In the gazebo launch file, spawn the controllers separately for each
robot, under a robotname namespace.

File: iiwa_description/urdf/iiwa14.urdf.xacro (robot description, xacro)
@@ -11,5 +11,8 @@
   <!--iiwa-->
   <xacro:iiwa14 hardware_interface="$(arg hardware_interface)" robot_name="$(arg robot_name)" parent="world">
-    <origin xyz="0 0 0.0" rpy="0 0 0" />
+    <origin xyz="1 1 0.0" rpy="0 0 0" />
+  </xacro:iiwa14>
+  <xacro:iiwa14 hardware_interface="$(arg hardware_interface)" robot_name="$(arg robot_name)2" parent="world">
+    <origin xyz="-1 -1 0.0" rpy="0 0 0" />
   </xacro:iiwa14>
 </robot>
