Commit message: Added missing dependency and added friction and ee_link rotation to urdf.

File: iiwa_description/urdf/iiwa14.xacro (robot description, xacro)
@@ -8,9 +8,10 @@
   <xacro:include filename="$(find iiwa_description)/urdf/utilities.xacro" />
   <!-- some constants -->
-  <xacro:property name="safety_controller_k_pos" value="100" />
-  <xacro:property name="safety_controller_k_vel" value="2" />
-  <xacro:property name="joint_damping" value="0.5" />
+  <xacro:property name="safety_controller_k_pos" value="100"/>
+  <xacro:property name="safety_controller_k_vel" value="2"/>
+  <xacro:property name="joint_damping" value="0.7"/>
+  <xacro:property name="friction" value="10.0"/>
   <xacro:property name="max_effort" value="300"/>
-  <xacro:property name="max_velocity" value="10"/>
+  <xacro:property name="max_velocity" value="1.0"/>
   <xacro:macro name="iiwa14" params="parent hardware_interface robot_name *origin">
     <!--joint between {parent} and link_0-->
@@ -59,5 +60,5 @@
                          k_position="${safety_controller_k_pos}"
                          k_velocity="${safety_controller_k_vel}"/>
-      <dynamics damping="${joint_damping}"/>
+      <dynamics damping="${joint_damping}" friction="${friction}"/>
     </joint>
     <link name="${robot_name}_link_1">
@@ -94,5 +95,5 @@
                          k_position="${safety_controller_k_pos}"
                          k_velocity="${safety_controller_k_vel}"/>
-      <dynamics damping="${joint_damping}"/>
+      <dynamics damping="${joint_damping}" friction="${friction}"/>
     </joint>
     <link name="${robot_name}_link_2">
@@ -129,5 +130,5 @@
                          k_position="${safety_controller_k_pos}"
                          k_velocity="${safety_controller_k_vel}"/>
-      <dynamics damping="${joint_damping}"/>
+      <dynamics damping="${joint_damping}" friction="${friction}"/>
     </joint>
     <link name="${robot_name}_link_3">
@@ -164,5 +165,5 @@
                          k_position="${safety_controller_k_pos}"
                          k_velocity="${safety_controller_k_vel}"/>
-      <dynamics damping="${joint_damping}"/>
+      <dynamics damping="${joint_damping}" friction="${friction}"/>
     </joint>
     <link name="${robot_name}_link_4">
@@ -199,5 +200,5 @@
                          k_position="${safety_controller_k_pos}"
                          k_velocity="${safety_controller_k_vel}"/>
-      <dynamics damping="${joint_damping}"/>
+      <dynamics damping="${joint_damping}" friction="${friction}"/>
     </joint>
     <link name="${robot_name}_link_5">
@@ -234,5 +235,5 @@
                          k_position="${safety_controller_k_pos}"
                          k_velocity="${safety_controller_k_vel}"/>
-      <dynamics damping="${joint_damping}"/>
+      <dynamics damping="${joint_damping}" friction="${friction}"/>
     </joint>
     <link name="${robot_name}_link_6">
@@ -269,5 +270,5 @@
                          k_position="${safety_controller_k_pos}"
                          k_velocity="${safety_controller_k_vel}"/>
-      <dynamics damping="${joint_damping}"/>
+      <dynamics damping="${joint_damping}" friction="${friction}"/>
     </joint>
     <link name="${robot_name}_link_7">
@@ -295,5 +296,5 @@
       <parent link="${robot_name}_link_7"/>
       <child link="${robot_name}_link_ee"/>
-      <origin xyz="0 0 0.045" rpy="0 0 0"/>
+      <origin xyz="0 0 0.045" rpy="0 -${PI/2} 0"/>
     </joint>
     <link name="${robot_name}_link_ee">
