Commit message: Properly fixed installation and headers of various files.

File: iiwa_description/urdf/iiwa7.xacro (robot description, xacro)
@@ -10,7 +10,7 @@
   <xacro:property name="safety_controller_k_pos" value="100" />
   <xacro:property name="safety_controller_k_vel" value="2" />
-  <xacro:property name="joint_damping" value="0.5" />
+  <xacro:property name="joint_damping" value="1.0" />
   <xacro:property name="max_effort" value="300"/>
-  <xacro:property name="max_velocity" value="10"/>
+  <xacro:property name="max_velocity" value="0.5"/>
   <xacro:macro name="iiwa7" params="parent hardware_interface robot_name *origin">
     <!--joint between {parent} and link_0-->
